File: hardware/PCB/Click4/Click4.kicad_pcb (KiCad board)
At the start: 2 copper layers, 44.9 x 71.1 mm, 65 parts, among them J1 USB_C_Receptacle_USB2.0_16P, Q1 MMBT3904_C181119, SW1 SK-3296S-01-L3, U1 PCF8563TS, U14 RP2354A, U2 AP2112K-3.3, U3 KLJ-5030-5040, U5 ETA6003Q3Q_C5455585, Y1 Crystal, Y2 Crystal

Commit message: correct pcb folder
Parts:
- moved Y2 1.14 mm to (177.8, 108.5), turned to 0 degrees
- moved C36 0.49 mm to (160.8, 109.4)
Routing:
- net GND: track 11.6 -> 25.0 mm, vias 5 -> 695
- net +3V3: track 182.4 -> 187.7 mm
- net /SDA: track 96.7 -> 101.9 mm
- net /SCL: track 88.9 -> 93.1 mm
- net Vol_Dvd: track 74.9 -> 77.1 mm
- net /GPIO1: track 57.2 -> 59.1 mm
- net Net-(U1-OSCI): track 6.28 -> 4.55 mm
- net /SYS: track 93.9 -> 92.3 mm, vias 5 -> 6
- net +BATT: track 39.3 -> 40.6 mm
- net VBUS_USB: track 29.4 -> 30.5 mm
- net Net-(U1-OSCO): track 7.80 -> 6.89 mm
- net +1V1: track 24.8 -> 24.3 mm
- net /BUZZER: vias 3 -> 2
- added copper zone on B.Cu, net GND
- added copper zone on F.Cu, net GND
