File: hardware/PCB/Click4/Click4.kicad_pcb (KiCad board)
At the start: 2 copper layers, 44.9 x 71.1 mm, 65 parts, among them J1 USB_C_Receptacle_USB2.0_16P, Q1 MMBT3904_C181119, SW1 SK-3296S-01-L3, U1 PCF8563TS, U14 RP2354A, U2 AP2112K-3.3, U3 KLJ-5030-5040, U5 ETA6003Q3Q_C5455585, Y1 Crystal, Y2 Crystal

Commit message: leaderboard management and stats syncing
Parts:
- added C43: 1uF, Capacitor_SMD:C_0603_1608Metric, F.Cu at (147.8, 62.8)
- added C44: 1uF, Capacitor_SMD:C_0603_1608Metric, F.Cu at (187.6, 61.9)
- added TP1: TestPoint, TestPoint:TestPoint_Pad_D1.0mm, B.Cu at (165.8, 101.8)
- added TP10: TestPoint, TestPoint:TestPoint_Pad_D1.0mm, F.Cu at (167.7, 66.7)
- added TP11: TestPoint, TestPoint:TestPoint_Pad_D1.0mm, F.Cu at (158.0, 73.2)
- added TP12: TestPoint, TestPoint:TestPoint_Pad_D1.0mm, F.Cu at (160.6, 71.7)
- added TP13: TestPoint, TestPoint:TestPoint_Pad_D1.0mm, F.Cu at (183.9, 97.6)
- added TP14: TestPoint, TestPoint:TestPoint_Pad_D1.0mm, B.Cu at (158.0, 73.2)
- added TP15: TestPoint, TestPoint:TestPoint_Pad_D1.0mm, F.Cu at (147.9, 76.5)
- added TP16: TestPoint, TestPoint:TestPoint_Pad_D1.0mm, F.Cu at (146.8, 79.5)
- added TP17: TestPoint, TestPoint:TestPoint_Pad_D1.0mm, B.Cu at (160.6, 71.7)
- added TP18: TestPoint, TestPoint:TestPoint_Pad_D1.0mm, B.Cu at (155.4, 96.5)
- added TP19: TestPoint, TestPoint:TestPoint_Pad_D1.0mm, B.Cu at (146.8, 79.5)
- added TP2: TestPoint, TestPoint:TestPoint_Pad_D1.0mm, B.Cu at (167.9, 103.0)
- added TP20: TestPoint, TestPoint:TestPoint_Pad_D1.0mm, B.Cu at (161.8, 52.5)
- added TP22: TestPoint, TestPoint:TestPoint_Pad_D1.0mm, F.Cu at (163.5, 56.0)
- added TP7: TestPoint, TestPoint:TestPoint_Pad_D1.0mm, B.Cu at (177.9, 47.3)
- added TP8: TestPoint, TestPoint:TestPoint_Pad_D1.0mm, F.Cu at (161.8, 52.5)
- added TP9: TestPoint, TestPoint:TestPoint_Pad_D1.0mm, F.Cu at (166.4, 64.2)
Routing:
- net GND: track 25.0 -> 37.0 mm, vias 695 -> 273
- net /SYS: track 92.3 -> 97.5 mm
- net +3V3: track 187.7 -> 192.2 mm
- net Net-(J1-CC2): track 2.86 -> 7.09 mm
- net +1V1: track 24.3 -> 26.7 mm
- net VBUS_USB: track 30.5 -> 32.5 mm, vias 4 -> 5
- net +BATT: track 40.6 -> 40.1 mm
- net Net-(D4-CKI): track 50.2 -> 50.5 mm, vias 0 -> 1
- net Net-(D3-CKI): track 60.3 -> 60.4 mm, vias 2 -> 3
- net Net-(D4-SDI): vias 0 -> 1
- net Net-(D3-SDI): vias 2 -> 3

Commit message: PCB LED changes and simple re-routing
Parts:
- removed C43, C44: 1uF, Capacitor_SMD:C_0603_1608Metric
- removed D3, D4: APA102-2020, LED_SMD:LED-APA102-2020
- removed L2: L, Resistor_SMD:R_0805_2012Metric
- removed TP11, TP12, TP14, TP15, TP16, TP19: TestPoint, TestPoint:TestPoint_Pad_D1.0mm
- added C45: 1uF, Capacitor_SMD:C_0603_1608Metric, F.Cu at (151.8, 60.1)
- added C46: 1uF, Capacitor_SMD:C_0603_1608Metric, F.Cu at (187.2, 62.4)
- added L1: AOTA-B201610S3R3-101-T, easyeda2kicad:IND-SMD_L2.0-W1.6_AOTA-B201610S3R3-101-T, F.Cu at (170.2, 106.4)
- added LED1: XL-2020RGBC-WS2812B, easyeda2kicad:LED-SMD_4P-L2.0-W2.0-BR-1, F.Cu at (149.0, 59.4)
- added LED2: XL-2020RGBC-WS2812B, easyeda2kicad:LED-SMD_4P-L2.0-W2.0-BR-1, F.Cu at (186.5, 59.4)
- moved TP18 48.2 mm to (188.2, 61.2)
- moved TP17 17.3 mm to (146.8, 61.2)
- moved BT1 0.50 mm to (151.7, 66.6)
Connections:
- TP17 pad 1: Net-(D3-SDI) -> /DI
- TP18 pad 1: Net-(D4-CKI) -> Net-(LED1-DO)
- U14 pad 15: Net-(D4-CKI) -> /DI
- U14 pad 16: Net-(D4-SDI) -> unconnected-(U14-GPIO12-Pad16)
Routing:
- net Net-(LED1-DO): track 0.00 -> 65.7 mm, vias 0 -> 3
- net Net-(D3-SDI): track 60.6 -> 0.00 mm, vias 3 -> 0
- net Net-(D3-CKI): track 60.4 -> 0.00 mm, vias 3 -> 0
- net Net-(D4-SDI): track 51.8 -> 0.00 mm, vias 1 -> 0
- net Net-(D4-CKI): track 50.5 -> 0.00 mm, vias 1 -> 0
- net /DI: track 0.00 -> 49.8 mm, vias 0 -> 1
- net +3V3: track 192.2 -> 190.7 mm
- net GND: track 37.0 -> 36.0 mm, vias 273 -> 271
