File: hardware/PCB/Click4/Click4.kicad_pcb (KiCad board)
At the start: 2 copper layers, 44.9 x 71.1 mm, 78 parts, among them J1 USB_C_Receptacle_USB2.0_16P, Q1 MMBT3904_C181119, SW1 SK-3296S-01-L3, U1 PCF8563TS, U14 RP2354A, U2 AP2112K-3.3, U3 KLJ-5030-5040, U5 ETA6003Q3Q_C5455585, Y1 Crystal, Y2 Crystal

Commit message: PCB LED Updates
Parts:
- LED1, LED2: value XL-2020RGBC-WS2812B -> SK6812SIDE-A_C5378721; footprint easyeda2kicad:LED-SMD_4P-L2.0-W2.0-BR-1 -> easyeda2kicad:LED-SMD_4P-L4.0-W1.6-L
- moved C46 4.27 mm to (184.4, 59.1), turned to 0 degrees
- moved TP18 2.75 mm to (188.7, 64.0)
- moved C45 1.84 mm to (150.1, 60.8), turned to 90 degrees
- moved TP17 1.50 mm to (146.8, 62.8)
- moved LED1 1.49 mm to (147.5, 59.5)
- moved LED2 1.03 mm to (187.5, 59.5), turned to -90 degrees
Connections:
- LED1 pad 1: Net-(LED1-DO) -> /DI
- LED1 pad 2: GND -> +3V3
- LED1 pad 3: /DI -> Net-(LED1-DOUT)
- LED1 pad 4: +3V3 -> GND
- LED2 pad 1: unconnected-(LED2-DO-Pad1) -> Net-(LED1-DOUT)
- LED2 pad 2: GND -> +3V3
- LED2 pad 3: Net-(LED1-DO) -> unconnected-(LED2-DOUT-Pad3)
- LED2 pad 4: +3V3 -> GND
- TP18 pad 1: Net-(LED1-DO) -> Net-(LED1-DOUT)
Routing:
- net Net-(LED1-DOUT): track 0.00 -> 68.1 mm, vias 0 -> 3
- net Net-(LED1-DO): track 65.7 -> 0.00 mm, vias 3 -> 0
- net GND: track 36.0 -> 40.1 mm, vias 269 -> 266
- net /DI: track 49.8 -> 48.0 mm
- net +3V3: track 189.7 -> 188.2 mm
