File: hardware/PCB/Click4/Click4.kicad_sch (KiCad schematic)
At the start: 67 parts, among them J1 USB_C_Receptacle_USB2.0_16P, J3 OLED_128x64, Q1 MMBT3904_C181119, SW1 SK-3296S-01-L3, U1 PCF8563TS, U14 RP2354A, U2 AP2112K-3.3, U3 KLJ-5030-5040, U5 ETA6003Q3Q_C5455585, Y1 Crystal, Y2 Crystal

Commit message: leaderboard management and stats syncing
Parts:
- added C43, C44: 1uF, Capacitor_SMD:C_0603_1608Metric, symbol easyeda2kicad:TCC0603X7R105K250CT
- added TP1, TP10, TP11, TP12, TP13, TP14, TP15, TP16, TP17, TP18, TP19, TP2, TP20, TP22, TP7, TP8, TP9: TestPoint, TestPoint:TestPoint_Pad_D1.0mm, symbol Connector:TestPoint
Connections:
- net +3V3: now also C43.2, C44.2
- net GND: now also C43.1, C44.1
- net SCL: now also TP2.1
- net SDA: now also TP1.1
- net SYS: now also TP13.1, TP7.1
- net USB_DN: now also TP10.1
- net USB_DP: now also TP9.1
- net VBUS_USB: now also TP20.1, TP8.1
- net at D3.4 (SDI), D4.3 (SDO): now also TP12.1, TP17.1
- net at D3.5 (CKI), D4.2 (CKO): now also TP11.1, TP14.1
- net at J1.B5 (CC2), R52.1: now also TP22.1
- net at D4.5 (CKI), U14.15 (GPIO11): now also TP15.1, TP18.1
- net at D4.4 (SDI), U14.16 (GPIO12): now also TP16.1, TP19.1

Commit message: PCB LED changes and simple re-routing
Parts:
- removed C43, C44: 1uF, Capacitor_SMD:C_0603_1608Metric, symbol easyeda2kicad:TCC0603X7R105K250CT
- removed D3, D4: APA102-2020, LED_SMD:LED-APA102-2020, symbol LED:APA102-2020
- removed L2: L, Resistor_SMD:R_0805_2012Metric, symbol Device:L
- removed TP11, TP12, TP14, TP15, TP16, TP19: TestPoint, TestPoint:TestPoint_Pad_D1.0mm, symbol Connector:TestPoint
- added C45, C46: 1uF, Capacitor_SMD:C_0603_1608Metric, symbol easyeda2kicad:TCC0603X7R105K250CT
- added L1: AOTA-B201610S3R3-101-T, easyeda2kicad:IND-SMD_L2.0-W1.6_AOTA-B201610S3R3-101-T, symbol easyeda:AOTA-B201610S3R3-101-T
- added LED1, LED2: XL-2020RGBC-WS2812B, easyeda2kicad:LED-SMD_4P-L2.0-W2.0-BR-1, symbol easyeda:XL-2020RGBC-WS2812B
- C25, C26, C29: LCSC Part (none) -> C23733
- C27, C28, C30, C31, C34, C35, C36, C37, C38, C39, C40, C41: LCSC Part (none) -> C1525
- C33: LCSC Part (none) -> C19666; MPN (none) -> CL10A475KO8NNNC
- C42: LCSC Part (none) -> C15525
- J1: LCSC Part (none) -> C2765186
- J3, S1, S2, TP1, TP10, TP13, TP17, TP18, TP2, TP20, TP22, TP3, TP4, TP5, TP6, TP7, TP8, TP9: now not fitted; now left out of the parts list
- R1, R2: LCSC Part (none) -> C25744
- R23, R50, R51: LCSC Part (none) -> C138002
- R4: LCSC Part (none) -> C21190; MPN (none) -> RT0603FRE101KL
- R49, R54, R55: LCSC Part (none) -> C21190
- R52, R53: LCSC Part (none) -> C25905
- U1: LCSC Part (none) -> C27397
- Y1: LCSC Part (none) -> C20625731
- Y2: LCSC Part (none) -> C97604
Connections:
- net +1V1: now also L1.1
- net +3V3: now also C45.2, C46.2, LED1.4 (VDD), LED2.4 (VDD)
- net GND: now also C45.1, C46.1, LED1.2 (GND), LED2.2 (GND)
- net VREG_LX: now also L1.2
- net at TP18.1: now also LED1.1 (DO), LED2.3 (DI); no longer U14.15 (GPIO11)
- net DI: now reaches TP17.1
- net DI: now also U14.15 (GPIO11), LED1.3 (DI)

Commit message: PCB LED Updates
Parts:
- removed LED1, LED2: XL-2020RGBC-WS2812B, easyeda2kicad:LED-SMD_4P-L2.0-W2.0-BR-1, symbol easyeda:XL-2020RGBC-WS2812B
- added LED1, LED2: SK6812SIDE-A_C5378721, easyeda2kicad:LED-SMD_4P-L4.0-W1.6-L, symbol easyeda:SK6812SIDE-A_C5378721
Connections:
- net +3V3: now also LED1.2 (VDD), LED2.2 (VDD)
- net DI: now also LED1.1 (DIN)
- net GND: now also LED1.4 (GND), LED2.4 (GND)
- net at TP18.1: now also LED1.3 (DOUT), LED2.1 (DIN)
Other:
- moved on the sheet: C25, C26, C27, C28, C29, C30, C33, C34, C35, C36, C37, C38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
